File: r2/src/safeproject-led-r2.kicad_pcb (KiCad board)
At the start: 2 copper layers, 29 x 51.5 mm, 20 parts, among them J1 2842142-4, J2 FH12-20S-0.5SH

Commit message: Add 200 to all designators to prevent collisoins in the panel
Parts:
- R207: renamed from R7; value 100R -> 22R
- R208: renamed from R8; value 100R -> 22R
- R209: renamed from R9; value 100R -> 22R
- renumbered J1 to J201, J2 to J202, LED1 to LED201, LED2 to LED202, LED3 to LED203, R1 to R201, R2 to R202, R3 to R203, R4 to R204, R5 to R205, R6 to R206

Commit message: Update PCB with hole names
Parts:
- H205, H206: renamed from ?; value (none) -> MountingHole
- renumbered REF** to H201, REF** to H202, REF** to H203, REF** to H204
Changed lines of the file:
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@@
   (footprint "" locked (layer "F.Cu")
     (at 4.5 -9)
-    (fp_text reference "" (at 0 0) (layer "F.SilkS")
+    (property "Sheetfile" "safeproject-led-r2.kicad_sch")
+    (property "Sheetname" "")
+    (fp_text reference "H205" (at 0 0) (layer "F.SilkS") hide
       (effects (font (size 1.27 1.27) (thickness 0.15)))
     )
-    (fp_text value "" (at 0 0) (layer "F.SilkS")
+    (fp_text value "MountingHole" (at 0 0) (layer "F.SilkS") hide
       (effects (font (size 1.27 1.27) (thickness 0.15)))
     )
@@
   (footprint "" locked (layer "F.Cu")
     (at 0 35.5)
-    (fp_text reference "" (at 0 0) (layer "F.SilkS")
+    (property "Sheetfile" "safeproject-led-r2.kicad_sch")
+    (property "Sheetname" "")
+    (fp_text reference "H206" (at 0 0) (layer "F.SilkS") hide
       (effects (font (size 1.27 1.27) (thickness 0.15)))
     )
-    (fp_text value "" (at 0 0) (layer "F.SilkS")
+    (fp_text value "MountingHole" (at 0 0) (layer "F.SilkS") hide
       (effects (font (size 1.27 1.27) (thickness 0.15)))
     )
@@
     (descr "Mounting Hole 3.2mm, no annular, M3, DIN965")
     (tags "mounting hole 3.2mm no annular m3 din965")
-    (attr exclude_from_pos_files exclude_from_bom)
-    (fp_text reference "REF**" (at 0 -3.8) (layer "F.SilkS") hide
+    (property "Sheetfile" "safeproject-led-r2.kicad_sch")
+    (property "Sheetname" "")
+    (attr exclude_from_pos_files)
+    (fp_text reference "H204" (at 0 -3.8) (layer "F.SilkS") hide
       (effects (font (size 1 1) (thickness 0.15)))
     )
@@
     (descr "Mounting Hole 3.2mm, no annular, M3, DIN965")
     (tags "mounting hole 3.2mm no annular m3 din965")
-    (attr exclude_from_pos_files exclude_from_bom)
-    (fp_text reference "REF**" (at 0 -3.8) (layer "F.SilkS") hide
+    (property "Sheetfile" "safeproject-led-r2.kicad_sch")
+    (property "Sheetname" "")
+    (attr exclude_from_pos_files)
+    (fp_text reference "H201" (at 0 -3.8) (layer "F.SilkS") hide
       (effects (font (size 1 1) (thickness 0.15)))
     )
@@
     (descr "Mounting Hole 3.2mm, no annular, M3, DIN965")
     (tags "mounting hole 3.2mm no annular m3 din965")
+    (property "Sheetfile" "safeproject-led-r2.kicad_sch")
+    (property "Sheetname" "")
     (clearance 1.4)
     (zone_connect 0)
-    (attr exclude_from_pos_files exclude_from_bom)
-    (fp_text reference "REF**" (at 0 -3.8) (layer "F.SilkS") hide
+    (attr exclude_from_pos_files)
+    (fp_text reference "H203" (at 0 -3.8) (layer "F.SilkS") hide
       (effects (font (size 1 1) (thickness 0.15)))
     )
@@
     (descr "Mounting Hole 3.2mm, no annular, M3, DIN965")
     (tags "mounting hole 3.2mm no annular m3 din965")
-    (attr exclude_from_pos_files exclude_from_bom)
-    (fp_text reference "REF**" (at 0 -3.8) (layer "F.SilkS") hide
+    (property "Sheetfile" "safeproject-led-r2.kicad_sch")
+    (property "Sheetname" "")
+    (attr exclude_from_pos_files)
+    (fp_text reference "H202" (at 0 -3.8) (layer "F.SilkS") hide
       (effects (font (size 1 1) (thickness 0.15)))
     )
