File: r4/src/bugg-led-r4.kicad_pcb (KiCad board)
At the start: 2 copper layers, 29 x 51.5 mm, 22 parts, among them J201 2314844-8, J202 FH12A-20S-0.5SH

Commit message: Update footprints. Fix missing soldermask cutouts in mounting holes
Parts:
- H201, H202, H203, H204: footprint MountingHole:MountingHole_3.2mm_M3_DIN965 -> jeffmakes-footprints:MountingHole_3.2mm_M3_DIN965_no_soldermask
- R201, R202, R203: value 22R -> 22k
- R204, R205, R206: value 22R -> 39k
- R207, R208, R209: value 22R -> 10k
Other:
- copper layers 2 -> 6

Commit message: Change submodule settings so, hopefully, submodules don't get into a detatched-head state (https://stackoverflow.com/questions/7124486/what-to-do-with-commit-made-in-a-detached-head)
Parts:
- H205, H206: footprint (none) -> jeffmakes-footprints:MountingHole_2.0mm
Routing:
- added copper zone on In1.Cu, net GND
- added copper zone on In2.Cu, net GND
- added copper zone on In3.Cu, net GND
- added copper zone on In4.Cu, net GND
Other:
- board text added: "bugg-led-r4 Monad 2022"
- board text removed: "bugg-led-r3 Monad 2021"
