File: r5/src/bugg-led-r5.kicad_sch (KiCad schematic)
At the start: 22 parts, among them J201 2314844-8, J202 FH12A-20S-0.5SH

Commit message: Replace board-to-board connector with type with alignment pegs
Parts:
- J201: footprint jeffmakes-footprints:PinSocket_2x04_P2.00mm_Vertical_SMD_Bottom_or_Top_Entry_AMPMODU -> jeffmakes-footprints:BF100-08-A-C-1-0625-L-C

Commit message: DRC pass
Parts:
- J201: value 2314844-8 -> BF100-08-A-C-1-0625-L-C
Changed lines of the file:
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@@
       (effects (font (size 1.27 1.27)) (justify left))
     )
-    (property "Value" "2314844-8" (at 171.45 85.09 0)
+    (property "Value" "BF100-08-A-C-1-0625-L-C" (at 171.45 85.09 0)
       (effects (font (size 1.27 1.27)) (justify left))
     )

Commit message: Change all resistors to 0402. Update symbols and footprints to those in latest libraries.
Parts:
- R201, R202, R203, R204, R205, R206, R207, R208, R209: footprint Resistor_SMD:R_0603_1608Metric -> Resistor_SMD:R_0402_1005Metric

Commit message: Additional BoM info. Fabrication data exported automatically with lacKi
Parts:
- J201: MPN (none) -> BF100-08-A-C-1-0625-L-C; Manufacturer (none) -> GCT; Mouser (none) -> 640-BF108AC10625LC
- J202: Digikey (none) -> HFK120CT-ND; MPN (none) -> FH12A-20S-0.5SH(55); Manufacturer (none) -> Hirose; Mouser (none) -> 798-FH12A-20S0.5SH55
- LED201, LED202, LED203: Digikey (none) -> 1830-1116-6-ND; MPN (none) -> IN-P32TATRGB; Manufacturer (none) -> Inolux; Mouser (none) -> 743-IN-P32TATRGB
